File: nrf52board.sch (KiCad schematic (older format))
At the start: 9 parts

Commit message: added board symbol
Parts:
- added U1: nrf52board, symbol nrf52:nrf52board
- gave numbers to parts that had none: 9
Connections:
- net labels added: +5V, P0.02, P0.03, P0.04, P0.05, P0.06, P0.07, P0.08, P0.09, P0.10, P0.11, P0.12, P0.13, P0.14, P0.15, P0.16, P0.17, P0.18, P0.19, P0.20, P0.21, P0.22, P0.23, P0.24, P0.25, P0.26, P0.27, P0.28, P0.29, P0.30, P0.31
- wire segments 41 -> 107

Commit message: moved libs to kicad-libs
Parts:
- added C?: 4.7u, symbol Device:C
- added J?: USB_B_Micro, symbol Connector_Specialized:USB_B_Micro
- added JP? (x6): SolderJumper_2_Open, symbol Jumper:SolderJumper_2_Open
- added R?: R, symbol Device:R
- added R?: 1M, symbol Device:R
- added U?: RFM95W-868S2, symbol RF_AM_FM:RFM95W-868S2
Connections:
- net labels added: D+, D-, DIO0, DIO1, DIO2, DIO3, DIO4, DIO5, MISO, MOSI, NSS_LORA, RESET_LORA, SCK
- wire segments 107 -> 144
- no-connect marks 0 -> 2

Commit message: sch: added power
Parts:
- added C? (x2): 1u, symbol Device:C
- added C?: 0.01u, symbol Device:C
- added C? (x2): 4.7u, symbol Device:C
- added D?: LED, symbol Device:LED
- added D?: D_Schottky, symbol Device:D_Schottky
- added J?: Battery, symbol Connector_Generic:Conn_01x02
- added Q?: Q_PMOS_DSG, symbol Device:Q_PMOS_DSG
- added R?: 470, symbol Device:R
- added R?: 100k, symbol Device:R
- added U?: MCP73831-2-OT, Package_TO_SOT_SMD:SOT-23-5, symbol Battery_Management:MCP73831-2-OT
- added U?: LP2985-3.3, Package_TO_SOT_SMD:SOT-23-5, symbol Regulator_Linear:LP2985-3.3
Connections:
- net labels added: +3.3V, +BATT
- wire segments 144 -> 188

Commit message: charger done
Parts:
- removed C?: 0.01u, symbol Device:C
- added R?: 10k, symbol Device:R
Connections:
- wire segments 188 -> 190
- no-connect marks 2 -> 3
Other:
- note added: "10k = 100 mA charge"
- note added: "Actual PN LP5907MFX-3.3/NOPB"
- note added: "TODO:\n- add cp2103\n- match LoRa to NRF\n- add buttons\n- add LEDs"
Changed lines of the file:
@@
 	5550 2300 5450 2300
 NoConn ~ 6050 1350
-Text GLabel 4950 1350 0    50   Input ~ 0
-SCK
 Text GLabel 4950 1450 0    50   Input ~ 0
 MOSI
@@
 	1    0    0    -1
 $EndComp
-$Comp
-L Device:C C?
-U 1 1 5ADAE27F
-P 5150 3850
-F 0 "C?" H 5265 3896 50  0000 L CNN
-F 1 "0.01u" H 5265 3805 50  0000 L CNN
-F 2 "" H 5188 3700 50  0001 C CNN
-F 3 "~" H 5150 3850 50  0001 C CNN
-	1    5150 3850
-	1    0    0    -1
-$EndComp
-Wire Wire Line
-	5050 3700 5150 3700
 Wire Wire Line
 	5150 4000 5150 4050
@@
 L power:GND #PWR?
 U 1 1 5ADE9DC5
-P 1450 5950
-F 0 "#PWR?" H 1450 5700 50  0001 C CNN
-F 1 "GND" H 1455 5777 50  0000 C CNN
-F 2 "" H 1450 5950 50  0001 C CNN
-F 3 "" H 1450 5950 50  0001 C CNN
-	1    1450 5950
-	1    0    0    -1
-$EndComp
-Wire Wire Line
-	1450 5850 1450 5900
+P 1450 6300
+F 0 "#PWR?" H 1450 6050 50  0001 C CNN
+F 1 "GND" H 1455 6127 50  0000 C CNN
+F 2 "" H 1450 6300 50  0001 C CNN
+F 3 "" H 1450 6300 50  0001 C CNN
+	1    1450 6300
+	1    0    0    -1
+$EndComp
+Wire Wire Line
+	1450 5850 1450 6250
 $Comp
 L Device:LED D?
@@
 $EndComp
 Wire Wire Line
-	850  5550 850  5900
-Wire Wire Line
-	850  5900 1450 5900
-Connection ~ 1450 5900
-Wire Wire Line
-	1450 5900 1450 5950
+	850  5550 850  6250
+Wire Wire Line
+	850  6250 1050 6250
+Connection ~ 1450 6250
+Wire Wire Line
+	1450 6250 1450 6300
 Wire Wire Line
 	1450 5150 850  5150
@@
 	2850 5450 2850 5750
 Wire Wire Line
-	2850 5850 2850 5900
-Wire Wire Line
-	1450 5900 2450 5900
-Wire Wire Line
-	2450 5850 2450 5900
-Connection ~ 2450 5900
-Wire Wire Line
-	2450 5900 2850 5900
+	1450 6250 2450 6250
+Wire Wire Line
+	2450 5850 2450 6250
+Connection ~ 2450 6250
+Wire Wire Line
+	2450 6250 2850 6250
 $Comp
 L power:+BATT #PWR?
@@
 	3250 3600 3350 3600
 Connection ~ 3350 3600
+Text GLabel 4950 1350 0    50   Input ~ 0
+SCK
+NoConn ~ 5050 3700
+Text Notes 4150 3300 0    50   ~ 0
+Actual PN LP5907MFX-3.3/NOPB
+Text Notes 8100 4900 0    50   ~ 0
+TODO:\n- add cp2103\n- match LoRa to NRF\n- add buttons\n- add LEDs
+$Comp
+L Device:R R?
+U 1 1 5AFDF948
+P 1050 5950
+F 0 "R?" V 843 5950 50  0000 C CNN
+F 1 "10k" V 934 5950 50  0000 C CNN
+F 2 "" V 980 5950 50  0001 C CNN
+F 3 "~" H 1050 5950 50  0001 C CNN
+	1    1050 5950
+	-1   0    0    1
+$EndComp
+Wire Wire Line
+	2850 5850 2850 6250
+Wire Wire Line
+	1050 5650 1050 5800
+Wire Wire Line
+	1050 6100 1050 6250
+Connection ~ 1050 6250
+Wire Wire Line
+	1050 6250 1450 6250
+Text Notes 1500 6050 0    50   ~ 0
+10k = 100 mA charge
 $EndSCHEMATC

Commit message: sch: update todo
Other:
- note added: "TODO:\n- add cp2103\n- match LoRa to NRF\n- add buttons\n- add LEDs\n- add LoRa IPX/UFL"
- note removed: "TODO:\n- add cp2103\n- match LoRa to NRF\n- add buttons\n- add LEDs"
Changed lines of the file:
@@
 Wire Wire Line
 	5550 2300 5450 2300
-NoConn ~ 6050 1350
 Text GLabel 4950 1450 0    50   Input ~ 0
 MOSI
@@
 Actual PN LP5907MFX-3.3/NOPB
 Text Notes 8100 4900 0    50   ~ 0
-TODO:\n- add cp2103\n- match LoRa to NRF\n- add buttons\n- add LEDs
+TODO:\n- add cp2103\n- match LoRa to NRF\n- add buttons\n- add LEDs\n- add LoRa IPX/UFL
 $Comp
 L Device:R R?
@@
 Text Notes 1500 6050 0    50   ~ 0
 10k = 100 mA charge
+NoConn ~ 6050 1350
 $EndSCHEMATC

Commit message: sch: updated TODO
Connections:
- wire segments 190 -> 188
Other:
- note added: "TODO:\n- add cp2103\n- RX/TX as in DK\n- RTS/CTS to RESET/DEBUG\n- match LoRa to NRF\n- add buttons as in DK\n- add LEDs as in DK\n- add LoRa IPX/UFL"
- note removed: "TODO:\n- add cp2103\n- match LoRa to NRF\n- add buttons\n- add LEDs\n- add LoRa IPX/UFL"
Changed lines of the file:
@@
 	1    0    0    -1
 $EndComp
-Wire Wire Line
-	5150 4000 5150 4050
-Wire Wire Line
-	5150 4050 4650 4050
 $Comp
 L power:+3.3V #PWR?
@@
 Wire Wire Line
 	5550 3900 5550 4050
-Wire Wire Line
-	5550 4050 5150 4050
-Connection ~ 5150 4050
 Wire Wire Line
 	1850 5450 2450 5450
@@
 Actual PN LP5907MFX-3.3/NOPB
 Text Notes 8100 4900 0    50   ~ 0
-TODO:\n- add cp2103\n- match LoRa to NRF\n- add buttons\n- add LEDs\n- add LoRa IPX/UFL
+TODO:\n- add cp2103\n- RX/TX as in DK\n- RTS/CTS to RESET/DEBUG\n- match LoRa to NRF\n- add buttons as in DK\n- add LEDs as in DK\n- add LoRa IPX/UFL
 $Comp
 L Device:R R?
@@
 10k = 100 mA charge
 NoConn ~ 6050 1350
+Wire Wire Line
+	4650 4050 5550 4050
 $EndSCHEMATC

Commit message: sch: added cp2102, lora connected
Parts:
- added C? (x2): 0.1u, symbol Device:C
- added C?: 1u, symbol Device:C
- added D?: LED, symbol Device:LED
- added JP?: SolderJumper_2_Open, symbol Jumper:SolderJumper_2_Open
- added R? (x2): 10k, symbol Device:R
- added R?: 1k, symbol Device:R
- added SW?: SW_Push, symbol Switch:SW_Push
- added U?: CP2102-GM, QFN28, symbol usb-uart:CP2102-GM
- R?: value R -> 10k
Connections:
- net labels removed: DIO0, DIO1, DIO2, DIO3, DIO4, DIO5, MISO, MOSI, NSS_LORA, SCK
- wire segments 188 -> 229
- no-connect marks 3 -> 7
Other:
- note added: "TODO:\n- add USB ESD\n- add LoRa IPX/UFL"
- note removed: "TODO:\n- add cp2103\n- RX/TX as in DK\n- RTS/CTS to RESET/DEBUG\n- match LoRa to NRF\n- add buttons as in DK\n- add LEDs as in DK\n- add LoRa IPX/UFL"

Commit message: sch: added one more btn and led
Parts:
- added D?: LED, LED_SMD:LED_0603_1608Metric, symbol Device:LED
- added R?: 1k, Resistor_SMD:R_0603_1608Metric, symbol Device:R
- added SW?: SW_Push, Button_Switch_SMD:Panasonic_EVQPUJ_EVQPUA, symbol Switch:SW_Push
- C1, C2, C3, C4, C5: footprint (none) -> Capacitor_SMD:C_0603_1608Metric
- C10, C11, C12, C13, C6, C7, C8, C9: renamed from C?; footprint (none) -> Capacitor_SMD:C_0603_1608Metric
- D1, D3: renamed from D?; footprint (none) -> LED_SMD:LED_0603_1608Metric
- D2: renamed from D?; footprint (none) -> Diode_SMD:D_SOD-323
- J1: footprint (none) -> Connector_PinHeader_2.54mm:PinHeader_1x04_P2.54mm_Vertical
- J2: renamed from J?; footprint (none) -> Connector_USB:USB_Micro-B_Amphenol_10103594-0001LF_Horizontal
- J3: renamed from J?; footprint (none) -> Connector_PinHeader_2.54mm:PinHeader_1x02_P2.54mm_Vertical
- JP1, JP2, JP3, JP4, JP5, JP6, JP7: renamed from JP?; footprint (none) -> Jumper:SolderJumper-2_P1.3mm_Open_RoundedPad1.0x1.5mm
- L1, L2: footprint (none) -> Inductor_SMD:L_0805_2012Metric
- Q1: renamed from Q?; footprint (none) -> Package_TO_SOT_SMD:SOT-23
- R1, R2, R3, R4, R5, R6, R7, R8: renamed from R?; footprint (none) -> Resistor_SMD:R_0603_1608Metric
- SW1: renamed from SW?; footprint (none) -> Button_Switch_SMD:Panasonic_EVQPUJ_EVQPUA
- U1: footprint (none) -> nrf52:nrf52board
- U2: footprint (none) -> nrf52:E73-2G4M04S
- U5: renamed from U?; footprint (none) -> RF_Module:Hopref_RFM9XW_SMD
- U6: renamed from U?; footprint QFN28 -> Package_DFN_QFN:QFN-28-1EP_5x5mm_P0.5mm_EP3.35x3.35mm
- gave numbers to parts that had none: 2
Connections:
- net labels removed: RESET_LORA
- wire segments 229 -> 242
